File: hardware/KICAD Projects/Single side S3 temp sense/Single side S3 temp sense.kicad_sch (KiCad schematic)
At the start: 40 parts, among them J1 TYPE-C-31-M-12, J2 DTF13-6P, SW1 PTS810_SJM_250_SMTR_LFS, SW2 PTS810_SJM_250_SMTR_LFS, U1 AMS1117-3.3, U2 ESP32-S3-WROOM-1, U3 MCP2515-I, U4 TJA1050DRG, X1 ${ALTIUM_VALUE}

Commit message: nfkljasdnfl
Parts:
- removed UNIT_1: ARDUINO_NANO, BAJA SAE:SHIELD_ARDUINO_NANO, symbol BAJA SAE:ARDUINO_NANO
Other:
- moved on the sheet: C1, C10, C2, C3, C4, C5, C6, C7, C8, C9, D1, D2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

Commit message: finished the single side temp sense
Parts:
- removed C11: 10uF/16V, Capacitor_Tantalum_SMD:CP_EIA-1608-08_AVX-J, symbol CAN Integration-altium-import:root_0_Cap_Tantalum_adafruit.IntLib
- removed C15: ${ALTIUM_VALUE}, Capacitor_SMD:C_0603_1608Metric, symbol CAN Integration-altium-import:root_2_Cap_0603_adafruit.IntLib
- removed D6: SK6812, LED_SMD:LED_SK6812_PLCC4_5.0x5.0mm_P3.2mm, symbol LED:SK6812
- removed U2: ESP32-S3-WROOM-1, RF_Module:ESP32-S3-WROOM-1, symbol RF_Module:ESP32-S3-WROOM-1
- added C16, C17: 100n, Capacitor_SMD:C_0603_1608Metric, symbol Device:C
- added C18, C19: 1u, Capacitor_SMD:C_0603_1608Metric, symbol Device:C
- added C20: 10u, Capacitor_SMD:C_0603_1608Metric, symbol Device:C
- added C21, C22: 10pf, Capacitor_SMD:C_0603_1608Metric, symbol Device:C
- added R10, R11: 4.7K, Resistor_SMD:R_0201_0603Metric, symbol Device:R
- added R12: 10k, Resistor_SMD:R_0201_0603Metric, symbol Device:R
- added R13, R14, R15: 22, Resistor_SMD:R_0201_0603Metric, symbol Device:R
- added R7: 33, Resistor_SMD:R_0201_0603Metric, symbol Device:R
- added S1: PESD2CAN_215, 0_Custom:DIO_PESD2CAN_215, symbol 0_Custom:PESD2CAN_215
- added U2: ESP32-S3FN8, 0_Custom:IC_ESP32-S3, symbol 0_Custom:ESP32-S3
- added U6: USBLC6-2SC6, Package_TO_SOT_SMD:SOT-23-6, symbol Power_Protection:USBLC6-2SC6
- added X2: ${ALTIUM_VALUE}, Crystal:Crystal_SMD_HC49-SD, symbol CAN Integration-altium-import:root_0_CRYSTAL-ECS-100-20-5PVX_adafruit.IntLib
- C6: value 1u -> 100n
- C7: value 10u -> 100n
- C8: value 0u1 -> 100n
- R4, R9: value 10k -> 33; footprint Resistor_SMD:R_0603_1608Metric -> Resistor_SMD:R_0201_0603Metric
Connections:
- net 0: now also C6.1, C7.1, C8.1, J2.3, C16.1, C17.1, C18.1, C19.1, C20.1, C21.2, C22.2, S1.3, U2.57 (GND), U6.2 (GND); no longer C6.2, C7.2, C8.2, J2.2
- net CHIP_PU: now also U2.4 (CHIP_PU); no longer C6.1, R4.2
- net CS: now also R12.2, U2.19 (GPIO14)
- net D+: now also U6.3 (I/O2)
- net D-: now also U6.1 (I/O1)
- net GPI00: now also U2.5 (GPIO0)
- net High: now also J2.2, J2.5, S1.2; no longer J2.4, J2.6
- net Low: now also J2.1, J2.6, S1.1; no longer J2.3, J2.5
- net SCK: now also R7.1
- net SCL: now also R11.1, U2.15 (GPIO10)
- net SDA: now also R10.2, U2.14 (GPIO9)
- net SI: now also R4.1
- net SO: now also R9.1
- net VCC: now also J2.4, U6.5 (VBUS); no longer J2.1
- net VCC_3V3: now also C6.2, C7.2, C8.2, C16.2, C17.2, C18.2, C19.2, C20.2, R10.1, R11.2, R12.1, U2.20 (VDD3P3_RTC), U2.29 (VDD_SPI), U2.46 (VDD3P3_CPU), U2.55 (VDDA1), U2.56 (VDDA2); no longer C7.1, C8.1, R9.2
- removed net ESP_3V3: R4.1, R9.1
- new net: C21.1, R15.2, X2.1
- new net: R14.1, U6.4 (I/O2)
- new net: R14.2, U2.26 (GPIO20)
- new net: R7.2, U2.16 (GPIO11)
- new net: R4.2, U2.17 (GPIO12)
- new net: R9.2, U2.18 (GPIO13)
- new net: U2.2 (VDD3P3), U2.3 (VDD3P3)
- new net: R13.1, U2.25 (GPIO19)
- new net: R13.2, U6.6 (I/O1)
- new net XTAL_N: C22.1, U2.53 (XTAL_N), X2.2
- new net XTAL_P: R15.1, U2.54 (XTAL_P)
- no-connect marks 32 -> 47
Other:
- note added: "DO NOT USE"
- note added: "ESP-32 40MHZ Xtal"
- note added: "GPIO 0, 3, 45, 46 - Strapping pins (Boot Mode)"
- note added: "GPIO 30-32 if using onboard flash"
- note added: "Pull up resistors"
- note removed: "ESP-32"
- note removed: "I/O"
- note removed: "RGB LED"
- moved on the sheet: C1, C10, C2, C3, C4, C5, C9, D1, D2, D3, D4, D5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
